File: 2026/electric_vehicle/pcb/electric_vehicle_2026.kicad_sch (KiCad schematic)
At the start: 0 parts

Commit message: Write full code and schematic
Parts:
- added A1: Arduino_UNO_R3, Module:Arduino_UNO_R3, symbol MCU_Module:Arduino_UNO_R3
- added BT1: Battery-9V, symbol Device:Battery
- added M1: Motor_Servo, symbol Motor:Motor_Servo
- added SW1: SW_Push_Dual, symbol Switch:SW_Push_Dual
- added SW2: SW_SPDT, symbol Switch:SW_SPDT
Connections:
- new net: A1.29 (GND), M1.3 (-), SW1.1, SW2.2 (B)
- new net: A1.22 (D7), SW1.4
- new net: A1.24 (D9), M1.1 (PWM)
- new net: A1.5 (+5V), M1.2 (+)
- new net: A1.23 (D8), SW2.3 (C)
- new net: A1.7 (GND), BT1.2 (-)
- new net: A1.8 (VIN), BT1.1 (+)
Other:
- note added: "note: goes to battery dc plug instead of VIN pin and GND pin"
- note added: "set INPUT_PULLUP"
